File: hardware/Electroencephalograph/EEGFrontendElectrode1To4.sch (KiCad schematic (older format))
At the start: 81 parts, among them J1 Conn_01x08_Male

Commit message: draft of PCB routing
Parts:
- renumbered C15 to C1, C6 to C10, C21 to C11, C17 to C12, C7 to C13, C22 to C14, C18 to C15, C2 to C16, C12 to C17, C19 to C18, C13 to C19, C4 to C2, C8 to C20, C14 to C21, C9 to C22, C3 to C23, C10 to C24, C23 to C3, C16 to C4, C24 to C6, C1 to C7, C11 to C8, C20 to C9, D12 to D10, D13 to D11, D15 to D12, D3 to D13, D4 to D14, D7 to D15, D10 to D16, D5 to D2, D8 to D3, D11 to D4, D14 to D5, D16 to D6, D2 to D7, D6 to D8, JP5 to JP2, JP8 to JP3, JP2 to JP4, JP6 to JP5, JP7 to JP6, JP3 to JP7, JP4 to JP8, R18 to R1, R23 to R10, R26 to R11, R32 to R12, R6 to R13, R27 to R14, R20 to R15, R7 to R16, R28 to R17, R21 to R18, R2 to R19, R4 to R2, R11 to R20, R15 to R21, R24 to R22, R25 to R23, R31 to R24, R16 to R25, R8 to R26, R17 to R27, R9 to R28, R3 to R29, R29 to R3, R12 to R30, R13 to R31, R22 to R32, R19 to R4, R30 to R6, R1 to R7, R10 to R8, R14 to R9
Connections:
- net labels added: ECC_1N, ECC_2N, ECC_3N, ECC_4N
- net labels removed: ECC_5P, ECC_6P, ECC_7P, ECC_8P
- wire segments 214 -> 216

Commit message: reshape power supply / acquisition
Parts:
- removed C16, C17, C18, C23, C24, C7, C8, C9: NC, Capacitor_SMD:C_0402_1005Metric, symbol Device:C
- removed JP1, JP2, JP3, JP4, JP5, JP6, JP7, JP8: Jumper_NO_Small, Jumper:SolderJumper-2_P1.3mm_Open_Pad1.0x1.5mm, symbol Device:Jumper_NO_Small
- added R83, R84, R85, R86, R87, R88, R89, R90: 0R, Resistor_SMD:R_0402_1005Metric, symbol Device:R
Connections:
- wire segments 216 -> 168
Other:
- moved on the sheet: R10, R11, R12, R19, R20, R21, R22, R23, R24, R29, R30, R31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
