File: hardware/Electroencephalograph/EEGFrontendElectrode5To8.sch (KiCad schematic (older format))
At the start: 81 parts, among them J2 Conn_01x08_Male

Commit message: draft of PCB routing
Parts:
- renumbered C86 to C70, C75 to C71, C94 to C72, C87 to C73, C76 to C74, C95 to C75, C72 to C76, C82 to C77, C91 to C78, C77 to C79, C92 to C80, C88 to C81, C78 to C82, C93 to C83, C89 to C84, C73 to C85, C83 to C86, C90 to C87, C84 to C88, C79 to C89, C85 to C90, C80 to C91, C74 to C92, C81 to C93, D25 to D22, D28 to D23, D31 to D24, D34 to D25, D36 to D26, D22 to D27, D26 to D28, D32 to D30, D33 to D31, D35 to D32, D23 to D33, D24 to D34, D27 to D35, D30 to D36, JP22 to JP25, JP29 to JP27, JP23 to JP28, JP27 to JP29, JP28 to JP30, JP24 to JP31, JP25 to JP32, R57 to R40, R43 to R41, R68 to R42, R58 to R43, R69 to R45, R40 to R46, R49 to R47, R53 to R48, R62 to R49, R65 to R50, R71 to R51, R45 to R52, R66 to R53, R59 to R54, R46 to R55, R67 to R56, R60 to R57, R41 to R58, R50 to R59, R54 to R60, R63 to R61, R64 to R62, R70 to R63, R55 to R64, R47 to R65, R56 to R66, R48 to R67, R42 to R68, R51 to R69, R52 to R70, R61 to R71
Connections:
- net labels added: ECC_5P, ECC_6P, ECC_7P, ECC_8P
- net labels removed: ECC_1N, ECC_2N, ECC_3N, ECC_4N
- wire segments 214 -> 216

Commit message: reshape power supply / acquisition
Parts:
- removed C76, C77, C78, C85, C86, C87, C92, C93: NC, Capacitor_SMD:C_0402_1005Metric, symbol Device:C
- removed JP25, JP26, JP27, JP28, JP29, JP30, JP31, JP32: Jumper_NO_Small, Jumper:SolderJumper-2_P1.3mm_Open_Pad1.0x1.5mm, symbol Device:Jumper_NO_Small
- added R91, R92, R93, R94, R95, R96, R97, R98: 0R, Resistor_SMD:R_0402_1005Metric, symbol Device:R
Connections:
- wire segments 216 -> 168
Other:
- moved on the sheet: R46, R47, R48, R49, R50, R51, R58, R59, R60, R61, R62, R63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
