File: Hardware/Electroencephalograph/DataProcessingPowerSupply.sch (KiCad schematic (older format))
At the start: 5 parts, among them J6 Conn_01x02_Female, U11 L78L33_SO8

Commit message: add bom
Parts:
- U11: symbol Regulator_Linear:L78L33_SO8 -> Electroencephalograph-rescue:L78L33_SO8-Regulator_Linear
Changed lines of the file:
@@
 $EndComp
 $Comp
-L Regulator_Linear:L78L33_SO8 U11
+L Electroencephalograph-rescue:L78L33_SO8-Regulator_Linear U11
 U 1 1 5ECE4DAC
 P 2700 3900
